File: pcb/nut-kb.kicad_pcb (KiCad board)
At the start: 2 copper layers, 65 parts, among them J1 Battery Connector, J2 E Ink Display, SW1 SW_Push, SW2 SW_SPST, U1 nice_nano

Commit message: [pcb] choc version done
Parts:
- added D31: D_Small, Diode_SMD:D_SOD-123, B.Cu at (95.0, 221.0)
- added D32: D_Small, Diode_SMD:D_SOD-123, B.Cu at (114.0, 219.0)
- added D33: D_Small, Diode_SMD:D_SOD-123, B.Cu at (133.0, 221.0)
- added D34: D_Small, Diode_SMD:D_SOD-123, B.Cu at (155.0, 224.0)
- added D35: D_Small, Diode_SMD:D_SOD-123, B.Cu at (171.0, 233.0)
- added D36: D_Small, Diode_SMD:D_SOD-123, B.Cu at (271.3, 151.6)
- added D37: D_Small, Diode_SMD:D_SOD-123, B.Cu at (290.3, 151.6)
- added D38: D_Small, Diode_SMD:D_SOD-123, B.Cu at (308.3, 146.9)
- added D39: D_Small, Diode_SMD:D_SOD-123, B.Cu at (328.3, 144.9)
- added D40: D_Small, Diode_SMD:D_SOD-123, B.Cu at (347.3, 146.9)
- added D41: D_Small, Diode_SMD:D_SOD-123, B.Cu at (366.3, 148.9)
- added D42: D_Small, Diode_SMD:D_SOD-123, B.Cu at (385.3, 148.9)
- added D43: D_Small, Diode_SMD:D_SOD-123, B.Cu at (271.3, 169.9)
- added D44: D_Small, Diode_SMD:D_SOD-123, B.Cu at (290.3, 169.9)
- added D45: D_Small, Diode_SMD:D_SOD-123, B.Cu at (308.3, 164.9)
- added D46: D_Small, Diode_SMD:D_SOD-123, B.Cu at (328.3, 162.9)
- added D47: D_Small, Diode_SMD:D_SOD-123, B.Cu at (347.3, 164.6)
- added D48: D_Small, Diode_SMD:D_SOD-123, B.Cu at (366.3, 166.9)
- added D49: D_Small, Diode_SMD:D_SOD-123, B.Cu at (385.3, 166.9)
- added D50: D_Small, Diode_SMD:D_SOD-123, B.Cu at (271.3, 187.9)
- added D51: D_Small, Diode_SMD:D_SOD-123, B.Cu at (290.3, 187.9)
- added D52: D_Small, Diode_SMD:D_SOD-123, B.Cu at (308.3, 182.9)
- added D53: D_Small, Diode_SMD:D_SOD-123, B.Cu at (328.3, 180.9)
- added D54: D_Small, Diode_SMD:D_SOD-123, B.Cu at (347.3, 182.6)
- added D55: D_Small, Diode_SMD:D_SOD-123, B.Cu at (366.3, 184.9)
- added D56: D_Small, Diode_SMD:D_SOD-123, B.Cu at (385.3, 184.9)
- added D57: D_Small, Diode_SMD:D_SOD-123, B.Cu at (271.3, 205.9)
- added D58: D_Small, Diode_SMD:D_SOD-123, B.Cu at (290.3, 205.9)
- added D59: D_Small, Diode_SMD:D_SOD-123, B.Cu at (308.3, 200.9)
- added D60: D_Small, Diode_SMD:D_SOD-123, B.Cu at (328.3, 198.9)
- added D61: D_Small, Diode_SMD:D_SOD-123, B.Cu at (347.3, 200.9)
- added D62: D_Small, Diode_SMD:D_SOD-123, B.Cu at (366.3, 202.9)
- added D63: D_Small, Diode_SMD:D_SOD-123, B.Cu at (385.3, 202.9)
- added D64: D_Small, Diode_SMD:D_SOD-123, B.Cu at (250.3, 230.9)
- added D65: D_Small, Diode_SMD:D_SOD-123, B.Cu at (266.3, 221.5)
- added D66: D_Small, Diode_SMD:D_SOD-123, B.Cu at (308.3, 218.9)
- added D67: D_Small, Diode_SMD:D_SOD-123, B.Cu at (328.3, 216.9)
- added D68: D_Small, Diode_SMD:D_SOD-123, B.Cu at (347.3, 218.9)
- added D69: D_Small, Diode_SMD:D_SOD-123, B.Cu at (366.3, 220.9)
- added D70: D_Small, Diode_SMD:D_SOD-123, B.Cu at (385.3, 220.9)
- added J3: E Ink Display, Connector_PinSocket_2.54mm:PinSocket_1x08_P2.54mm_Vertical, F.Cu at (236.4, 195.9)
- added J4: Battery Connector, Connector_JST:JST_PH_B3B-PH-K_1x03_P2.00mm_Vertical, F.Cu at (231.8, 181.0)
- added MX31: CMD, Switch_Keyboard_Kailh:SW_Kailh_Choc_V1_1.00u, F.Cu at (92.0, 217.3)
- added MX32: ??, Switch_Keyboard_Kailh:SW_Kailh_Choc_V1_1.00u, F.Cu at (111.0, 214.9)
- added MX33: ??, Switch_Keyboard_Kailh:SW_Kailh_Choc_V1_1.00u, F.Cu at (130.0, 217.3)
- added MX34: DELETE, Switch_Keyboard_Kailh:SW_Kailh_Choc_V1_2.00u_90deg, F.Cu at (157.0, 231.0)
- added MX35: SPACE, Switch_Keyboard_Kailh:SW_Kailh_Choc_V1_2.00u_90deg, F.Cu at (173.0, 240.0)
- added MX36: ??, Switch_Keyboard_Kailh:SW_Kailh_Choc_V1_1.00u, F.Cu at (267.7, 147.6)
- added MX37: #6, Switch_Keyboard_Kailh:SW_Kailh_Choc_V1_1.00u, F.Cu at (286.7, 147.6)
- added MX38: #7, Switch_Keyboard_Kailh:SW_Kailh_Choc_V1_1.00u, F.Cu at (305.7, 142.9)
- added MX39: #8, Switch_Keyboard_Kailh:SW_Kailh_Choc_V1_1.00u, F.Cu at (324.7, 140.5)
- added MX40: #9, Switch_Keyboard_Kailh:SW_Kailh_Choc_V1_1.00u, F.Cu at (343.7, 142.9)
- added MX41: #0, Switch_Keyboard_Kailh:SW_Kailh_Choc_V1_1.00u, F.Cu at (362.7, 145.3)
- added MX42: DELETE, Switch_Keyboard_Kailh:SW_Kailh_Choc_V1_1.00u, F.Cu at (381.7, 145.3)
- added MX43: ??, Switch_Keyboard_Kailh:SW_Kailh_Choc_V1_1.00u, F.Cu at (267.7, 165.6)
- added MX44: Y, Switch_Keyboard_Kailh:SW_Kailh_Choc_V1_1.00u, F.Cu at (286.7, 165.6)
- added MX45: U, Switch_Keyboard_Kailh:SW_Kailh_Choc_V1_1.00u, F.Cu at (305.7, 160.9)
- added MX46: I, Switch_Keyboard_Kailh:SW_Kailh_Choc_V1_1.00u, F.Cu at (324.7, 158.5)
- added MX47: O, Switch_Keyboard_Kailh:SW_Kailh_Choc_V1_1.00u, F.Cu at (343.7, 160.9)
- added MX48: P, Switch_Keyboard_Kailh:SW_Kailh_Choc_V1_1.00u, F.Cu at (362.7, 163.3)
- added MX49: |\, Switch_Keyboard_Kailh:SW_Kailh_Choc_V1_1.00u, F.Cu at (381.7, 163.3)
- added MX50: ??, Switch_Keyboard_Kailh:SW_Kailh_Choc_V1_1.00u, F.Cu at (267.7, 183.6)
- added MX51: H, Switch_Keyboard_Kailh:SW_Kailh_Choc_V1_1.00u, F.Cu at (286.7, 183.6)
- added MX52: J, Switch_Keyboard_Kailh:SW_Kailh_Choc_V1_1.00u, F.Cu at (305.7, 178.9)
- added MX53: K, Switch_Keyboard_Kailh:SW_Kailh_Choc_V1_1.00u, F.Cu at (324.7, 176.5)
- added MX54: L, Switch_Keyboard_Kailh:SW_Kailh_Choc_V1_1.00u, F.Cu at (343.7, 178.9)
- added MX55: ;, Switch_Keyboard_Kailh:SW_Kailh_Choc_V1_1.00u, F.Cu at (362.7, 181.3)
- added MX56: ', Switch_Keyboard_Kailh:SW_Kailh_Choc_V1_1.00u, F.Cu at (381.7, 181.3)
- added MX57: ??, Switch_Keyboard_Kailh:SW_Kailh_Choc_V1_1.00u, F.Cu at (267.7, 201.6)
- added MX58: N, Switch_Keyboard_Kailh:SW_Kailh_Choc_V1_1.00u, F.Cu at (286.7, 201.6)
- added MX59: M, Switch_Keyboard_Kailh:SW_Kailh_Choc_V1_1.00u, F.Cu at (305.7, 196.9)
- added MX60: <, Switch_Keyboard_Kailh:SW_Kailh_Choc_V1_1.00u, F.Cu at (324.7, 194.5)
- added MX61: >, Switch_Keyboard_Kailh:SW_Kailh_Choc_V1_1.00u, F.Cu at (343.7, 196.9)
- added MX62: ?, Switch_Keyboard_Kailh:SW_Kailh_Choc_V1_1.00u, F.Cu at (362.7, 199.3)
- added MX63: R_SHIFT, Switch_Keyboard_Kailh:SW_Kailh_Choc_V1_1.00u, F.Cu at (381.7, 199.3)
- added MX64: ??, Switch_Keyboard_Kailh:SW_Kailh_Choc_V1_2.00u_90deg, F.Cu at (262.3, 240.9)
- added MX65: ??, Switch_Keyboard_Kailh:SW_Kailh_Choc_V1_2.00u_90deg, F.Cu at (278.3, 231.9)
- added MX66: ??, Switch_Keyboard_Kailh:SW_Kailh_Choc_V1_1.00u, F.Cu at (305.7, 214.9)
- added MX67: ??, Switch_Keyboard_Kailh:SW_Kailh_Choc_V1_1.00u, F.Cu at (324.7, 212.5)
- added MX68: ??, Switch_Keyboard_Kailh:SW_Kailh_Choc_V1_1.00u, F.Cu at (343.7, 214.9)
- added MX69: ??, Switch_Keyboard_Kailh:SW_Kailh_Choc_V1_1.00u, F.Cu at (362.7, 217.3)
- added MX70: ??, Switch_Keyboard_Kailh:SW_Kailh_Choc_V1_1.00u, F.Cu at (381.7, 217.3)
- added REF**: breakaway-mousebites, random-keyboard-parts:breakaway-mousebites, F.Cu at (217.0, 166.1)
- added SW3: SW_Push, Button_Switch_THT:SW_PUSH_6mm, F.Cu at (232.3, 163.1)
- added SW4: SW_SPST, Button_Switch_THT:SW_DIP_SPSTx01_Slide_6.7x4.1mm_W7.62mm_P2.54mm_LowProfile, F.Cu at (225.2, 179.1)
- added U2: nice_nano_right, nice-nano-kicad:nice_nano, F.Cu at (245.3, 178.0)
- MX1, MX2, MX3, MX4, MX5, MX6: footprint MX_Only:MXOnly-1U-Hotswap-Antishear -> Switch_Keyboard_Kailh:SW_Kailh_Choc_V1_1.00u
- MX10: value E -> W; footprint MX_Only:MXOnly-1U-Hotswap-Antishear -> Switch_Keyboard_Kailh:SW_Kailh_Choc_V1_1.00u
- MX11: value R -> E; footprint MX_Only:MXOnly-1U-Hotswap-Antishear -> Switch_Keyboard_Kailh:SW_Kailh_Choc_V1_1.00u
- MX12: value T -> R; footprint MX_Only:MXOnly-1U-Hotswap-Antishear -> Switch_Keyboard_Kailh:SW_Kailh_Choc_V1_1.00u
- MX13: value ESC -> T; footprint MX_Only:MXOnly-1U-Hotswap-Antishear -> Switch_Keyboard_Kailh:SW_Kailh_Choc_V1_1.00u
- MX14: value A -> -; footprint MX_Only:MXOnly-1U-Hotswap-Antishear -> Switch_Keyboard_Kailh:SW_Kailh_Choc_V1_1.00u
- MX15: value S -> ESC; footprint MX_Only:MXOnly-1U-Hotswap-Antishear -> Switch_Keyboard_Kailh:SW_Kailh_Choc_V1_1.00u
- MX16: value D -> A; footprint MX_Only:MXOnly-1U-Hotswap-Antishear -> Switch_Keyboard_Kailh:SW_Kailh_Choc_V1_1.00u
- MX17: value F -> S; footprint MX_Only:MXOnly-1U-Hotswap-Antishear -> Switch_Keyboard_Kailh:SW_Kailh_Choc_V1_1.00u
- MX18: value G -> D; footprint MX_Only:MXOnly-1U-Hotswap-Antishear -> Switch_Keyboard_Kailh:SW_Kailh_Choc_V1_1.00u
- MX19: value SHIFT -> F; footprint MX_Only:MXOnly-1U-Hotswap-Antishear -> Switch_Keyboard_Kailh:SW_Kailh_Choc_V1_1.00u
- MX20: value Z -> G; footprint MX_Only:MXOnly-1U-Hotswap-Antishear -> Switch_Keyboard_Kailh:SW_Kailh_Choc_V1_1.00u
- MX21: value X -> [; footprint MX_Only:MXOnly-1U-Hotswap-Antishear -> Switch_Keyboard_Kailh:SW_Kailh_Choc_V1_1.00u
- MX22: value C -> L_SHIFT; footprint MX_Only:MXOnly-1U-Hotswap-Antishear -> Switch_Keyboard_Kailh:SW_Kailh_Choc_V1_1.00u
- MX23: value V -> Z; footprint MX_Only:MXOnly-1U-Hotswap-Antishear -> Switch_Keyboard_Kailh:SW_Kailh_Choc_V1_1.00u
- MX24: value B -> X; footprint MX_Only:MXOnly-1U-Hotswap-Antishear -> Switch_Keyboard_Kailh:SW_Kailh_Choc_V1_1.00u
- MX25: value CTRL -> C; footprint MX_Only:MXOnly-1U-Hotswap-Antishear -> Switch_Keyboard_Kailh:SW_Kailh_Choc_V1_1.00u
- MX26: value OPTION -> V; footprint MX_Only:MXOnly-1U-Hotswap-Antishear -> Switch_Keyboard_Kailh:SW_Kailh_Choc_V1_1.00u
- MX27: value CMD -> B; footprint MX_Only:MXOnly-1U-Hotswap-Antishear -> Switch_Keyboard_Kailh:SW_Kailh_Choc_V1_1.00u
- MX28: value MX-NoLED -> ??; footprint MX_Only:MXOnly-1U-Hotswap-Antishear -> Switch_Keyboard_Kailh:SW_Kailh_Choc_V1_1.00u
- MX29: value SPACE -> CTRL; footprint MX_Only:MXOnly-2U-Hotswap -> Switch_Keyboard_Kailh:SW_Kailh_Choc_V1_1.00u
- MX30: value LAYER1 -> OPTION; footprint MX_Only:MXOnly-2U-Hotswap -> Switch_Keyboard_Kailh:SW_Kailh_Choc_V1_1.00u
- MX7: value TAB -> ??; footprint MX_Only:MXOnly-1U-Hotswap-Antishear -> Switch_Keyboard_Kailh:SW_Kailh_Choc_V1_1.00u
- MX8: value Q -> TAB; footprint MX_Only:MXOnly-1U-Hotswap-Antishear -> Switch_Keyboard_Kailh:SW_Kailh_Choc_V1_1.00u
- MX9: value W -> Q; footprint MX_Only:MXOnly-1U-Hotswap-Antishear -> Switch_Keyboard_Kailh:SW_Kailh_Choc_V1_1.00u
- SW1: footprint Button_Switch_THT:SW_DIP_SPSTx01_Slide_6.7x4.1mm_W7.62mm_P2.54mm_LowProfile -> Button_Switch_THT:SW_PUSH_6mm
- U1: value nice_nano -> nice_nano_left
- moved MX7 172.8 mm to (168.0, 147.6)
- moved D7 169.0 mm to (171.0, 151.7)
- moved MX13 156.8 mm to (149.0, 165.6)
- moved MX14 156.8 mm to (168.0, 165.6)
- moved D13 153.4 mm to (152.0, 170.0)
- moved D14 153.3 mm to (171.0, 170.0)
- moved MX21 144.8 mm to (168.0, 183.6)
- moved MX20 141.6 mm to (149.0, 183.6)
- moved D21 141.6 mm to (171.0, 188.0)
- moved MX19 140.0 mm to (130.0, 181.3)
- moved D20 138.3 mm to (152.0, 188.0)
- moved D19 136.3 mm to (133.0, 185.0)
- moved J2 135.0 mm to (181.9, 196.0)
- moved U1 134.4 mm to (190.8, 178.0)
- moved MX28 132.8 mm to (168.0, 201.6)
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Connections:
- net +BATT renamed Net-(SW2-Pad1)
- net BUSY renamed L_BUSY
- net CLK renamed L_CLK
- net CS renamed L_CS
- net DC renamed L_DC
- net DIN renamed L_DIN
- net RESET renamed L_RESET
- net RST renamed L_RST
- D13 pad 1: ROW2 -> ROW1
- D14 pad 1: ROW2 -> ROW1
- D19 pad 1: ROW3 -> ROW2
- D20 pad 1: ROW3 -> ROW2
- D21 pad 1: ROW3 -> ROW2
- D25 pad 1: ROW4 -> ROW3
- D26 pad 1: ROW4 -> ROW3
- D27 pad 1: ROW4 -> ROW3
- D28 pad 1: ROW4 -> ROW3
- D7 pad 1: ROW1 -> ROW0
- MX10 pad 1: COL3 -> COL2
- MX11 pad 1: COL4 -> COL3
- MX12 pad 1: COL5 -> COL4
- MX13 pad 1: COL0 -> COL5
- MX14 pad 1: COL1 -> COL6
- MX15 pad 1: COL2 -> COL0
- MX16 pad 1: COL3 -> COL1
- MX17 pad 1: COL4 -> COL2
- MX18 pad 1: COL5 -> COL3
- MX19 pad 1: COL0 -> COL4
- MX20 pad 1: COL1 -> COL5
- MX21 pad 1: COL2 -> COL6
- MX22 pad 1: COL3 -> COL0
- MX23 pad 1: COL4 -> COL1
- MX24 pad 1: COL5 -> COL2
- MX25 pad 1: COL0 -> COL3
- MX26 pad 1: COL1 -> COL4
- MX27 pad 1: COL2 -> COL5
- MX28 pad 1: COL3 -> COL6
- MX29 pad 1: COL4 -> COL0
- MX30 pad 1: COL5 -> COL1
- MX7 pad 1: COL0 -> COL6
- MX8 pad 1: COL1 -> COL0
- MX9 pad 1: COL2 -> COL1
- U1 pad 11: ROW2 -> COL6
- U1 pad 12: ROW3 -> ROW2
- U1 pad 20: unconnected-(U1-Pad20) -> ROW3
Routing:
- net COL13: track 0.00 -> 214.5 mm
- net COL12: track 0.00 -> 196.2 mm
- net COL11: track 0.00 -> 176.9 mm
- net COL10: track 0.00 -> 157.6 mm
- net COL8: track 0.00 -> 143.6 mm
- net ROW9: track 0.00 -> 140.9 mm
- net COL9: track 0.00 -> 140.3 mm
- net COL6: track 0.00 -> 130.7 mm
- net COL7: track 0.00 -> 126.5 mm
- net ROW8: track 0.00 -> 118.6 mm
- net ROW7: track 0.00 -> 118.6 mm
- net ROW6: track 0.00 -> 118.6 mm
- net ROW5: track 0.00 -> 118.4 mm
- net GND1: track 0.00 -> 78.0 mm
- net ROW3: track 129.9 -> 171.8 mm
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Other:
- board outline added: 157.7 x 28.6 mm

Commit message: [pcb] finish keyboard
Parts:
- removed D36, D37, D38, D39, D40, D41, D42, D43, D44, D45, D46, D47, D48, D49, D50, D51, D52, D53, D54, D55, D56, D57, D58, D59, D60, D61, D62, D63, D64, D65, D66, D67, D68, D69, D70: D_Small, Diode_SMD:D_SOD-123
- removed J4: Battery Connector, Connector_JST:JST_PH_B3B-PH-K_1x03_P2.00mm_Vertical
- removed MX36, MX43, MX50, MX57, MX66, MX67, MX68, MX69, MX70: ??, Switch_Keyboard_Kailh:SW_Kailh_Choc_V1_1.00u
- removed MX37: #6, Switch_Keyboard_Kailh:SW_Kailh_Choc_V1_1.00u
- removed MX38: #7, Switch_Keyboard_Kailh:SW_Kailh_Choc_V1_1.00u
- removed MX39: #8, Switch_Keyboard_Kailh:SW_Kailh_Choc_V1_1.00u
- removed MX40: #9, Switch_Keyboard_Kailh:SW_Kailh_Choc_V1_1.00u
- removed MX41: #0, Switch_Keyboard_Kailh:SW_Kailh_Choc_V1_1.00u
- removed MX42: DELETE, Switch_Keyboard_Kailh:SW_Kailh_Choc_V1_1.00u
- removed MX44: Y, Switch_Keyboard_Kailh:SW_Kailh_Choc_V1_1.00u
- removed MX45: U, Switch_Keyboard_Kailh:SW_Kailh_Choc_V1_1.00u
- removed MX46: I, Switch_Keyboard_Kailh:SW_Kailh_Choc_V1_1.00u
- removed MX47: O, Switch_Keyboard_Kailh:SW_Kailh_Choc_V1_1.00u
- removed MX48: P, Switch_Keyboard_Kailh:SW_Kailh_Choc_V1_1.00u
- removed MX49: |\, Switch_Keyboard_Kailh:SW_Kailh_Choc_V1_1.00u
- removed MX51: H, Switch_Keyboard_Kailh:SW_Kailh_Choc_V1_1.00u
- removed MX52: J, Switch_Keyboard_Kailh:SW_Kailh_Choc_V1_1.00u
- removed MX53: K, Switch_Keyboard_Kailh:SW_Kailh_Choc_V1_1.00u
- removed MX54: L, Switch_Keyboard_Kailh:SW_Kailh_Choc_V1_1.00u
- removed MX55: ;, Switch_Keyboard_Kailh:SW_Kailh_Choc_V1_1.00u
- removed MX56: ', Switch_Keyboard_Kailh:SW_Kailh_Choc_V1_1.00u
- removed MX58: N, Switch_Keyboard_Kailh:SW_Kailh_Choc_V1_1.00u
- removed MX59: M, Switch_Keyboard_Kailh:SW_Kailh_Choc_V1_1.00u
- removed MX60: <, Switch_Keyboard_Kailh:SW_Kailh_Choc_V1_1.00u
- removed MX61: >, Switch_Keyboard_Kailh:SW_Kailh_Choc_V1_1.00u
- removed MX62: ?, Switch_Keyboard_Kailh:SW_Kailh_Choc_V1_1.00u
- removed MX63: R_SHIFT, Switch_Keyboard_Kailh:SW_Kailh_Choc_V1_1.00u
- removed MX64, MX65: ??, Switch_Keyboard_Kailh:SW_Kailh_Choc_V1_2.00u_90deg
- removed REF**: breakaway-mousebites, random-keyboard-parts:breakaway-mousebites
- removed SW3: SW_Push, Button_Switch_THT:SW_PUSH_6mm
- removed SW4: SW_SPST, Button_Switch_THT:SW_DIP_SPSTx01_Slide_6.7x4.1mm_W7.62mm_P2.54mm_LowProfile
- removed U2: nice_nano_right, nice-nano-kicad:nice_nano
- J2: value E Ink Display -> E Ink Display Left
- J3: value E Ink Display -> E Ink Display Right; moved to B.Cu
- MX1, MX10, MX11, MX12, MX13, MX14, MX15, MX16, MX17, MX18, MX19, MX2, MX20, MX21, MX22, MX23, MX24, MX25, MX26, MX27, MX28, MX29, MX3, MX30, MX31, MX32, MX33, MX4, MX5, MX6, MX7, MX8, MX9: footprint Switch_Keyboard_Kailh:SW_Kailh_Choc_V1_1.00u -> keyswitches:SW_PG1350_reversible
- MX34, MX35: footprint Switch_Keyboard_Kailh:SW_Kailh_Choc_V1_2.00u_90deg -> keyswitches:SW_PG1350_reversible
- U1: footprint nice-nano-kicad:nice_nano -> tairakb:nicenano
- moved J3 48.3 mm to (189.2, 185.6)
- moved SW1 35.0 mm to (177.0, 192.1), turned to -90 degrees
- moved J1 25.3 mm to (182.0, 197.0)
- moved SW2 24.7 mm to (188.4, 189.7)
- moved D35 21.6 mm to (151.2, 224.3), turned to 60 degrees
- moved D34 20.9 mm to (136.2, 214.9), turned to 60 degrees
- moved MX34 18.5 mm to (146.1, 216.0), turned to -30 degrees
- moved MX35 17.8 mm to (162.7, 225.5), turned to -30 degrees
- moved MX10 17.0 mm to (83.5, 148.5)
- moved MX12 17.0 mm to (121.5, 148.5)
- moved MX17 17.0 mm to (83.5, 166.5)
- moved MX19 17.0 mm to (121.5, 166.5)
- moved MX24 17.0 mm to (83.5, 184.5)
- moved MX26 17.0 mm to (121.5, 184.5)
- moved MX3 17.0 mm to (83.5, 130.5)
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Connections:
- net Net-(SW2-Pad1) renamed VCC
- J3 pad 1: R_CS -> L_CS
- J3 pad 2: R_DC -> L_DC
- J3 pad 3: GND1 -> GND
- J3 pad 5: R_CLK -> L_CLK
- J3 pad 6: R_DIN -> L_DIN
- J3 pad 7: R_RST -> L_RST
- J3 pad 8: R_BUSY -> L_BUSY
- U1 pad 10: COL5 -> L_CLK
- U1 pad 11: COL6 -> L_DIN
- U1 pad 12: ROW2 -> L_RST
- U1 pad 13: ROW4 -> L_BUSY
- U1 pad 14: L_BUSY -> COL0
- U1 pad 15: L_RST -> COL1
- U1 pad 16: L_DIN -> COL2
- U1 pad 17: L_CLK -> COL3
- U1 pad 18: L_DC -> COL4
- U1 pad 19: L_CS -> COL5
- U1 pad 20: ROW3 -> COL6
- U1 pad 5: COL0 -> ROW2
- U1 pad 6: COL1 -> ROW3
- U1 pad 7: COL2 -> ROW4
- U1 pad 8: COL3 -> L_DC
- U1 pad 9: COL4 -> L_CS
Routing:
- net COL13: track 214.5 -> 0.00 mm
- net COL12: track 196.2 -> 0.00 mm
- net COL11: track 176.9 -> 0.00 mm
- net COL10: track 157.6 -> 0.00 mm
- net COL8: track 143.6 -> 0.00 mm
- net ROW9: track 140.9 -> 0.00 mm
- net COL9: track 140.3 -> 0.00 mm
- net COL7: track 126.5 -> 0.00 mm
- net ROW8: track 118.6 -> 0.00 mm
- net ROW7: track 118.6 -> 0.00 mm
- net ROW6: track 118.6 -> 0.00 mm
- net ROW5: track 118.4 -> 0.00 mm
- net GND1: track 78.0 -> 0.00 mm
- net L_RESET: track 13.5 -> 70.1 mm
- net COL4: track 136.3 -> 179.9 mm
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Other:
- board size 157.7 x 28.6 mm -> 157 x 117 mm
